Commit message: 修改了urdf和sdf，让他更像真实场景

File: ros2_ws/src/my_arm_description/urdf/arm.urdf (robot description, URDF)
Before this commit: robot two_link_arm, 3 links, 2 joints
Links:
- removed link link1
- removed link link2
- added link cy1, mass 0.2; collision cylinder length=0.05 radius=0.1; visual cylinder length=0.05 radius=0.1
- added link cy3, mass 0.2; collision cylinder length=0.05 radius=0.1; visual cylinder length=0.05 radius=0.1
Joints:
- removed joint joint1
- removed joint joint2
- added joint joint3: type revolute, parent base_link, child cy1, origin xyz=0 0.25 0 rpy=1.5708 0 0, axis 0 1 0, limit lower=0 upper=0 effort=0 velocity=0
- added joint joint4: type revolute, parent base_link, child cy3, origin xyz=0 -0.25 0 rpy=1.5708 0 0, axis 0 -1 0, limit lower=0 upper=0 effort=0 velocity=0
